Commit message: add laser in xacro

File: mybot_description/urdf/kbot.xacro (robot description, xacro)
@@ -65,4 +65,18 @@
   <xacro:wheel prefix="left" reflect="1" />
   <xacro:wheel prefix="right" reflect="-1" />
+  <link name="laser_link">
+    <visual>
+      <origin xyz="0 0 0" rpy="0 0 0" />
+      <geometry>
+        <cylinder radius="${hokuyo_size}" length="0.04" />
+      </geometry>
+      <material name="blue" />
+    </visual>
+  </link>
+  <joint name="hokuyo_joint" type="fixed">
+    <origin xyz="0 0 ${base_height+hokuyo_size/4}" rpy="0 0 0" />
+    <parent link="base_link" />
+    <child link="laser_link" />
+  </joint>
   <!--
     <link name="camera">

File: mybot_description/urdf/properties.xacro (robot description, xacro)
@@ -17,5 +17,6 @@
    (currently in development and awaiting feedback)
 -->
-  <xacro:property name="gazebo" value="false" />
+  <xacro:property name="gazebo" value="true" />
+  <xacro:property name="hokuyo_size" value="0.03" />
   <xacro:property name="cam_px" value="-0.087" />
   <xacro:property name="cam_py" value="-0.0125" />
